File: hardware/main.kicad_sch (KiCad schematic)
At the start: 40 parts, among them J1 2.54-1*5P, J2 KH-2.54FH-1X2P-H8.5, U1 74HC595, U2 74HC595

Commit message: Updating from #1
Parts:
- D10, D11, D12, D13, D14, D15, D16, D17, D2, D3, D4, D5, D6, D7, D8, D9: lcsc C99772 -> C00000
Changed lines of the file:
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@@
 			)
 		)
-		(property "lcsc" "C99772"
+		(property "lcsc" "C00000"
 			(at 158.75 100.33 0)
 			(effects
@@
 			)
 		)
-		(property "lcsc" "C99772"
+		(property "lcsc" "C00000"
 			(at 158.75 46.99 0)
 			(effects
@@
 			)
 		)
-		(property "lcsc" "C99772"
+		(property "lcsc" "C00000"
 			(at 158.75 85.09 0)
 			(effects
@@
 			)
 		)
-		(property "lcsc" "C99772"
+		(property "lcsc" "C00000"
 			(at 158.75 62.23 0)
 			(effects
@@
 			)
 		)
-		(property "lcsc" "C99772"
+		(property "lcsc" "C00000"
 			(at 158.75 153.67 0)
 			(effects
@@
 			)
 		)
-		(property "lcsc" "C99772"
+		(property "lcsc" "C00000"
 			(at 158.75 146.05 0)
 			(effects
@@
 			)
 		)
-		(property "lcsc" "C99772"
+		(property "lcsc" "C00000"
 			(at 158.75 92.71 0)
 			(effects
@@
 			)
 		)
-		(property "lcsc" "C99772"
+		(property "lcsc" "C00000"
 			(at 158.75 115.57 0)
 			(effects
@@
 			)
 		)
-		(property "lcsc" "C99772"
+		(property "lcsc" "C00000"
 			(at 158.75 123.19 0)
 			(effects
@@
 			)
 		)
-		(property "lcsc" "C99772"
+		(property "lcsc" "C00000"
 			(at 158.75 77.47 0)
 			(effects
@@
 			)
 		)
-		(property "lcsc" "C99772"
+		(property "lcsc" "C00000"
 			(at 158.75 138.43 0)
 			(effects
@@
 			)
 		)
-		(property "lcsc" "C99772"
+		(property "lcsc" "C00000"
 			(at 158.75 39.37 0)
 			(effects
@@
 			)
 		)
-		(property "lcsc" "C99772"
+		(property "lcsc" "C00000"
 			(at 158.75 107.95 0)
 			(effects
@@
 			)
 		)
-		(property "lcsc" "C99772"
+		(property "lcsc" "C00000"
 			(at 158.75 54.61 0)
 			(effects
@@
 			)
 		)
-		(property "lcsc" "C99772"
+		(property "lcsc" "C00000"
 			(at 158.75 69.85 0)
 			(effects
@@
 			)
 		)
-		(property "lcsc" "C99772"
+		(property "lcsc" "C00000"
 			(at 158.75 130.81 0)
 			(effects
