File: hardware/main.kicad_sch (KiCad schematic)
At the start: 40 parts, among them J1 2.54-1*5P, J2 KH-2.54FH-1X2P-H8.5, U1 74HC595, U2 74HC595

Commit message: destroy pcb; fix sch
Connections:
- no-connect marks 1 -> 3
Changed lines of the file:
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@@
 		(at 123.19 123.19)
+	)
+	(no_connect
+		(at 44.45 127)
+	)
+	(no_connect
+		(at 44.45 124.46)
 	)
 	(wire

Commit message: Updating from #kici-example_stock_14560568212
Parts:
- C1, C2: pn (none) -> CC0805KRX7R9BB104
- D1: pn (none) -> 204-10SYGD/S530-E3
- D10, D11, D12, D13, D14, D15, D16, D17, D2, D3, D4, D5, D6, D7, D8, D9: pn (none) -> 204-10SURD/S530-A3
- J1: pn (none) -> 2.54-1*5P母
- J2: pn (none) -> KH-2.54FH-1X2P-H8.5
- R1, R10, R11, R12, R13, R14, R15, R16, R17, R2, R3, R4, R5, R6, R7, R8, R9: pn (none) -> 0805W8F4700T5E
- U1, U2: pn (none) -> 74HC595D
Changed lines of the file:
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@@
 			)
 		)
-		(property "pn" ""
+		(property "pn" "204-10SURD/S530-A3"
 			(at 158.75 100.33 0)
 			(effects
@@
 			)
 		)
-		(property "pn" ""
+		(property "pn" "74HC595D"
 			(at 113.03 49.53 0)
 			(effects
@@
 			)
 		)
-		(property "pn" ""
+		(property "pn" "204-10SURD/S530-A3"
 			(at 158.75 46.99 0)
 			(effects
@@
 			)
 		)
-		(property "pn" ""
+		(property "pn" "204-10SURD/S530-A3"
 			(at 158.75 85.09 0)
 			(effects
@@
 			)
 		)
-		(property "pn" ""
+		(property "pn" "204-10SURD/S530-A3"
 			(at 158.75 62.23 0)
 			(effects
@@
 			)
 		)
-		(property "pn" ""
+		(property "pn" "0805W8F4700T5E"
 			(at 149.86 115.57 0)
 			(effects
@@
 			)
 		)
-		(property "pn" ""
+		(property "pn" "0805W8F4700T5E"
 			(at 149.86 54.61 0)
 			(effects
@@
 			)
 		)
-		(property "pn" ""
+		(property "pn" "0805W8F4700T5E"
 			(at 149.86 69.85 0)
 			(effects
@@
 			)
 		)
-		(property "pn" ""
+		(property "pn" "204-10SYGD/S530-E3"
 			(at 45.72 93.98 0)
 			(effects
@@
 			)
 		)
-		(property "pn" ""
+		(property "pn" "0805W8F4700T5E"
 			(at 149.86 62.23 0)
 			(effects
@@
 			)
 		)
-		(property "pn" ""
+		(property "pn" "0805W8F4700T5E"
 			(at 45.72 86.36 0)
 			(effects
@@
 			)
 		)
-		(property "pn" ""
+		(property "pn" "204-10SURD/S530-A3"
 			(at 158.75 153.67 0)
 			(effects
@@
 			)
 		)
-		(property "pn" ""
+		(property "pn" "0805W8F4700T5E"
 			(at 149.86 77.47 0)
 			(effects
@@
 			)
 		)
-		(property "pn" ""
+		(property "pn" "0805W8F4700T5E"
 			(at 149.86 39.37 0)
 			(effects
@@
 			)
 		)
-		(property "pn" ""
+		(property "pn" "0805W8F4700T5E"
 			(at 149.86 123.19 0)
 			(effects
@@
 			)
 		)
-		(property "pn" ""
+		(property "pn" "204-10SURD/S530-A3"
 			(at 158.75 146.05 0)
 			(effects
@@
 			)
 		)
-		(property "pn" ""
+		(property "pn" "0805W8F4700T5E"
 			(at 149.86 107.95 0)
 			(effects
@@
 			)
 		)
-		(property "pn" ""
+		(property "pn" "204-10SURD/S530-A3"
 			(at 158.75 92.71 0)
 			(effects
@@
 			)
 		)
-		(property "pn" ""
+		(property "pn" "204-10SURD/S530-A3"
 			(at 158.75 115.57 0)
 			(effects
@@
 			)
 		)
-		(property "pn" ""
+		(property "pn" "0805W8F4700T5E"
 			(at 149.86 138.43 0)
 			(effects
@@
 			)
 		)
-		(property "pn" ""
+		(property "pn" "CC0805KRX7R9BB104"
 			(at 54.61 91.44 0)
 			(effects
@@
 			)
 		)
-		(property "pn" ""
+		(property "pn" "0805W8F4700T5E"
 			(at 149.86 153.67 0)
 			(effects
@@
 			)
 		)
-		(property "pn" ""
+		(property "pn" "204-10SURD/S530-A3"
 			(at 158.75 123.19 0)
 			(effects
@@
 			)
 		)
-		(property "pn" ""
+		(property "pn" "0805W8F4700T5E"
 			(at 149.86 46.99 0)
 			(effects
@@
 			)
 		)
-		(property "pn" ""
+		(property "pn" "204-10SURD/S530-A3"
 			(at 158.75 77.47 0)
 			(effects
@@
 			)
 		)
-		(property "pn" ""
+		(property "pn" "204-10SURD/S530-A3"
 			(at 158.75 138.43 0)
 			(effects
@@
 			)
 		)
-		(property "pn" ""
+		(property "pn" "CC0805KRX7R9BB104"
 			(at 63.5 91.44 0)
 			(effects
@@
 			)
 		)
-		(property "pn" ""
+		(property "pn" "204-10SURD/S530-A3"
 			(at 158.75 39.37 0)
 			(effects
@@
 			)
 		)
-		(property "pn" ""
+		(property "pn" "0805W8F4700T5E"
 			(at 149.86 130.81 0)
 			(effects
@@
 			)
 		)
-		(property "pn" ""
+		(property "pn" "204-10SURD/S530-A3"
 			(at 158.75 107.95 0)
 			(effects
@@
 			)
 		)
-		(property "pn" ""
+		(property "pn" "74HC595D"
 			(at 113.03 110.49 0)
 			(effects
@@
 			)
 		)
-		(property "pn" ""
+		(property "pn" "204-10SURD/S530-A3"
 			(at 158.75 54.61 0)
 			(effects
@@
 			)
 		)
-		(property "pn" ""
+		(property "pn" "0805W8F4700T5E"
 			(at 149.86 100.33 0)
 			(effects
@@
 			)
 		)
-		(property "pn" ""
+		(property "pn" "0805W8F4700T5E"
 			(at 149.86 146.05 0)
 			(effects
@@
 			)
 		)
-		(property "pn" ""
+		(property "pn" "204-10SURD/S530-A3"
 			(at 158.75 69.85 0)
 			(effects
@@
 			)
 		)
-		(property "pn" ""
+		(property "pn" "204-10SURD/S530-A3"
 			(at 158.75 130.81 0)
 			(effects
@@
 			)
 		)
-		(property "pn" ""
+		(property "pn" "0805W8F4700T5E"
 			(at 149.86 92.71 0)
 			(effects
@@
 			)
 		)
-		(property "pn" ""
+		(property "pn" "KH-2.54FH-1X2P-H8.5"
 			(at 49.53 124.46 0)
 			(effects
@@
 			)
 		)
-		(property "pn" ""
+		(property "pn" "2.54-1*5P母"
 			(at 63.5 39.37 0)
 			(effects
@@
 			)
 		)
-		(property "pn" ""
+		(property "pn" "0805W8F4700T5E"
 			(at 149.86 85.09 0)
 			(effects
